File: hd44780i2c.kicad_pcb (KiCad board)
At the start: 2 copper layers, 58.7 x 80.3 mm, 50 parts, among them J101 Conn_01x10_Female, J102 Conn_01x06_Female, J103 Conn_01x08_Female, J91 Conn_01x08_Female, Q1 BC337, Q2 2N7000, Q3 2N7000, SW1 SW_DIP_x01, SW11 SW_Push, SW21 SW_Push, SW31 SW_Push, SW41 SW_Push, SW51 SW_Push, U1 PCF8574A

Commit message: modifications
Parts:
- removed JP11, JP21, JP31, JP41, JP51: Jumper, Connector_PinHeader_2.54mm:PinHeader_1x03_P2.54mm_Vertical
- added RV2: 500, moja_biblioteka:Potentiometer_ACP_CA9-V5_Vertical, F.Cu at (30.9, 24.2)
- added SW2: SW_DIP_x05, Package_DIP:DIP-10_W7.62mm, F.Cu at (27.9, 97.8)
- Q1: footprint Package_TO_SOT_THT:TO-92_Inline -> Package_TO_SOT_THT:TO-92_Inline_Wide
- SW11: value SW_Push -> SW_SELECT
- SW21: value SW_Push -> SW_LEFT
- SW31: value SW_Push -> SW_UP
- SW41: value SW_Push -> SW_DOWN
- SW51: value SW_Push -> SW_RIGHT
- moved JP1 45.0 mm to (64.3, 60.5)
- moved JP2 45.0 mm to (64.3, 64.3)
- moved JP3 45.0 mm to (64.3, 68.1)
- moved REFL2 7.65 mm to (58.4, 54.6)
- moved RV1 7.62 mm to (41.1, 24.2)
- moved REFL3 5.71 mm to (64.8, 54.6)
- moved C51 5.12 mm to (53.4, 22.9)
- moved R52 5.08 mm to (55.9, 26.7)
- moved SW21 5.08 mm to (62.5, 50.2)
- moved SW51 5.08 mm to (62.5, 29.9)
- moved R51 5.08 mm to (45.7, 30.5)
- moved Q1 2.79 mm to (72.6, 91.1)
Connections:
- net Net-(C11-Pad1) renamed SELECT
- net Net-(R22-Pad1) renamed LEFT
- net Net-(R32-Pad1) renamed UP
- net Net-(R42-Pad1) renamed DOWN
- net Net-(R51-Pad2) renamed RIGHT
- DS1 pad 15: Net-(DS1-Pad15) -> Net-(DS1-LED(+))
- J91 pad 8: +3.3V -> unconnected-(J91-Pin_8-Pad8)
- SW1 pad 1: Net-(DS1-Pad15) -> Net-(RV2-Pad3)
Routing:
- net PB1: track 18.9 -> 148.6 mm
- net Net-(DS1-Pad15): track 72.8 -> 0.00 mm
- net Net-(DS1-LED(+)): track 0.00 -> 71.1 mm
- net PB4: track 13.6 -> 82.9 mm
- net D5: track 124.6 -> 56.0 mm
- net PB2: track 15.7 -> 77.5 mm
- net PB3: track 17.5 -> 70.9 mm
- net DOWN: track 53.4 -> 106.2 mm
- net SDAC: track 47.6 -> 94.2 mm
- net D4: track 54.5 -> 96.5 mm
- net PB0: track 48.0 -> 87.3 mm
- net GNDREF: track 270.0 -> 236.1 mm
- net Net-(JP1-C): track 12.6 -> 45.6 mm
- net Net-(DS1-VO): track 107.3 -> 139.9 mm
- net RIGHT: track 53.6 -> 84.8 mm
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- added copper zone on B.Cu, net GNDREF
Other:
- board text added: "5V/1"
- board text added: "BRIGHTNESS"
- board text added: "GND/0"
- board text added: "HD44780 I2C BOARD v2.0 Designed by Marcin Stodulski 2024 PINS 14-18 FOR BUTTONS ARE OPTIONALLY USED, DEPENDS ON JUMPERS SETTINGS U - MEANS PIN USED BY BOARD O/U - MEANS PIN OPTIONALLY USED BY BOARD 3V3 LOGIC"
- board text added: "SELECT to PB0"
- board text added: "Vin"
- board text added: "| switch to off | for programming"
- board text removed: "BTN"
- board text removed: "Button connected to"
- board text removed: "HD44780 I2C BOARD v1.0 Designed by M.S. 2023 I2C lines pulled up with logic level converter (3V3-5V)"
- board text removed: "PINS 14-18 FOR BUTTONS ARE OPTIONALLY USED, DEPENDS ON JUMPERS SETTINGS U - MEANS PIN USED BY BOARD O/U - MEANS PIN OPTIONALLY USED BY BOARD"
- board text removed: "SELECT button connected to PB0"
- board text removed: "UNCONNECTED"
- board text removed: "YES"
- board text removed: "| BTN UNCONNECTED"
