File: hd44780i2c.kicad_sch (KiCad schematic)
At the start: 47 parts, among them J101 Conn_01x10_Female, J102 Conn_01x06_Female, J103 Conn_01x08_Female, J91 Conn_01x08_Female, Q1 BC337, Q2 2N7000, Q3 2N7000, SW1 SW_DIP_x01, SW11 SW_Push, SW21 SW_Push, SW31 SW_Push, SW41 SW_Push, SW51 SW_Push, U1 PCF8574A

Commit message: modifications
Parts:
- removed JP11, JP21, JP31, JP41, JP51: Jumper, Connector_PinHeader_2.54mm:PinHeader_1x03_P2.54mm_Vertical, symbol Jumper:Jumper_3_Bridged12
- added RV2: 500, moja_biblioteka:Potentiometer_ACP_CA9-V5_Vertical, symbol Device:R_Potentiometer
- added SW2: SW_DIP_x05, Package_DIP:DIP-10_W7.62mm, symbol Switch:SW_DIP_x05
- J101: symbol Connector:Conn_01x10_Female -> Connector:Conn_01x10_Socket
- J102: symbol Connector:Conn_01x06_Female -> Connector:Conn_01x06_Socket
- J103, J91: symbol Connector:Conn_01x08_Female -> Connector:Conn_01x08_Socket
- Q1: footprint Package_TO_SOT_THT:TO-92_Inline -> Package_TO_SOT_THT:TO-92_Inline_Wide
- RV1: footprint Potentiometer_THT:Potentiometer_ACP_CA9-V10_Vertical -> moja_biblioteka:Potentiometer_ACP_CA9-V5_Vertical
- SW11: value SW_Push -> SW_SELECT
- SW21: value SW_Push -> SW_LEFT
- SW31: value SW_Push -> SW_UP
- SW41: value SW_Push -> SW_DOWN
- SW51: value SW_Push -> SW_RIGHT
Connections:
- net +3.3V: no longer J91.8 (Pin_8)
- net GNDREF: now also RV2.1
- net PB0: now also SW2.10
- net PB1: now also SW2.9
- net PB2: now also SW2.8
- net PB3: now also SW2.7
- net PB4: now also SW2.6
- net UP: now reaches C31.1, R31.2, R32.1
- net UP: now also SW2.3
- net SELECT: now reaches C11.1, R11.2, R12.1
- net SELECT: now also SW2.1
- net LEFT: now reaches C21.1, R21.2, R22.1
- net LEFT: now also SW2.2
- net RIGHT: now reaches C51.1, R51.2, R52.1
- net RIGHT: now also SW2.5
- net at DS1.15 (LED(+)): now also RV2.2; no longer SW1.1
- net DOWN: now reaches C41.1, R41.2, R42.1
- net DOWN: now also SW2.4
- new net: RV2.3, SW1.1
- no-connect marks 26 -> 22
Other:
- moved on the sheet: SW1
